Commit message: feat: change input dev name

File: models/rby1a/model.urdf (robot description, URDF)
Before this commit: robot RB_Y1_V1.0.1, 31 links, 30 joints
Joints:
- joint torso_2: limit lower=-2.44346095 upper=1.570796 effort=1000.0 velocity=3.14159265 -> lower=-2.617993 upper=1.570796 effort=1000.0 velocity=3.14159265

Commit message: feat: urdf update

File: models/rby1a/model.urdf (robot description, URDF)
Before this commit: robot RB_Y1_V1.0.1, 31 links, 30 joints
Joints:
- joint torso_2: limit lower=-2.617993 upper=1.570796 effort=1000.0 velocity=3.14159265 -> lower=-2.478367 upper=1.570796 effort=1000.0 velocity=3.14159265

Commit message: model update

File: models/rby1a/model.urdf (robot description, URDF)
Before this commit: robot RB_Y1_V1.0.1, 31 links, 30 joints
Links:
- link link_left_arm_0: geometry collision capsule length=0.0700 radius=0.075; visual mesh filename=./meshes/LINK_14.stl
- link link_left_arm_1: geometry collision capsule length=0.2000 radius=0.050; visual mesh filename=./meshes/LINK_15.stl
- link link_left_arm_2: geometry collision capsule length=0.080000 radius=0.05; visual mesh filename=./meshes/LINK_16.stl
- link link_left_arm_3: geometry collision capsule length=0.1150 radius=0.04; visual mesh filename=./meshes/LINK_17.stl
- link link_left_arm_4: geometry collision capsule length=0.095000 radius=0.035; visual mesh filename=./meshes/LINK_18.stl
- link link_left_arm_5: geometry collision capsule length=0.052000 radius=0.075; visual mesh filename=./meshes/LINK_19.stl
- link link_right_arm_0: geometry collision capsule length=0.0700 radius=0.075; visual mesh filename=./meshes/LINK_7.stl
- link link_right_arm_1: geometry collision capsule length=0.2000 radius=0.050; visual mesh filename=./meshes/LINK_8.stl
- link link_right_arm_2: geometry collision capsule length=0.080000 radius=0.05; visual mesh filename=./meshes/LINK_9.stl
- link link_right_arm_3: geometry collision capsule length=0.1150 radius=0.04; visual mesh filename=./meshes/LINK_10.stl
- link link_right_arm_4: geometry collision capsule length=0.095000 radius=0.035; visual mesh filename=./meshes/LINK_11.stl
- link link_right_arm_5: geometry collision capsule length=0.052000 radius=0.075; visual mesh filename=./meshes/LINK_12.stl
- link link_torso_0: geometry collision capsule length=0.230 radius=0.105; visual mesh filename=./meshes/LINK_1.stl
- link link_torso_1: geometry collision capsule length=0.220 radius=0.115; visual mesh filename=./meshes/LINK_2.stl
- link link_torso_2: geometry collision capsule length=0.1600 radius=0.095; visual mesh filename=./meshes/LINK_3.stl
- link link_torso_4: geometry collision capsule length=0.2 radius=0.105; visual mesh filename=./meshes/LINK_5.stl
- link link_torso_5: geometry collision capsule length=0.1350 radius=0.155; visual mesh filename=./meshes/LINK_6.stl

Commit message: update

File: models/rby1a/model.urdf (robot description, URDF)
Before this commit: robot RB_Y1_V1.0.1, 31 links, 30 joints
Links:
- link link_left_arm_1: geometry collision capsule colaffinity=768 length=0.2000 radius=0.050; visual mesh filename=./meshes/LINK_15.stl
- link link_left_arm_2: geometry collision capsule colaffinity=768 length=0.080000 radius=0.05; visual mesh filename=./meshes/LINK_16.stl
- link link_left_arm_3: geometry collision capsule colaffinity=926 length=0.1150 radius=0.04; visual mesh filename=./meshes/LINK_17.stl
- link link_left_arm_4: geometry collision capsule colaffinity=1022 length=0.095000 radius=0.035; visual mesh filename=./meshes/LINK_18.stl
- link link_left_arm_5: geometry collision capsule colaffinity=1023 length=0.052000 radius=0.075; visual mesh filename=./meshes/LINK_19.stl
- link link_right_arm_1: geometry collision capsule coltype=32 length=0.2000 radius=0.050; visual mesh filename=./meshes/LINK_8.stl
- link link_right_arm_2: geometry collision capsule coltype=64 length=0.080000 radius=0.05; visual mesh filename=./meshes/LINK_9.stl
- link link_right_arm_3: geometry collision capsule colaffinity=30 coltype=128 length=0.1150 radius=0.04; visual mesh filename=./meshes/LINK_10.stl
- link link_right_arm_4: geometry collision capsule colaffinity=30 coltype=256 length=0.095000 radius=0.035; visual mesh filename=./meshes/LINK_11.stl
- link link_right_arm_5: geometry collision capsule colaffinity=31 coltype=512 length=0.052000 radius=0.075; visual mesh filename=./meshes/LINK_12.stl
- link link_torso_0: geometry collision capsule coltype=1 length=0.230 radius=0.105; visual mesh filename=./meshes/LINK_1.stl
- link link_torso_1: geometry collision capsule coltype=2 length=0.220 radius=0.115; visual mesh filename=./meshes/LINK_2.stl
- link link_torso_2: geometry collision capsule coltype=4 length=0.1600 radius=0.095; visual mesh filename=./meshes/LINK_3.stl
- link link_torso_4: geometry collision capsule coltype=8 length=0.2 radius=0.105; visual mesh filename=./meshes/LINK_5.stl
- link link_torso_5: geometry collision capsule coltype=16 length=0.1350 radius=0.155; visual mesh filename=./meshes/LINK_6.stl
