Commit message: model update

File: models/rby1m/urdf/model.urdf (robot description, URDF)
Before this commit: robot RB_Y1M, 36 links, 35 joints
Links:
- link base: mass 60.08042639 -> 82.93082168
- link wheel_fl_link: mass 1.37783736 -> 2.54417879; geometry visual mesh filename=./meshes/MECANUM_WHEEL.dae
- link wheel_fr_link: mass 1.37783736 -> 2.54410022; geometry visual mesh filename=./meshes/MECANUM_WHEEL.dae
- link wheel_rl_link: mass 1.37783736 -> 2.54417879; geometry visual mesh filename=./meshes/MECANUM_WHEEL_M.dae
- link wheel_rr_link: mass 1.37783736 -> 2.54410022; geometry visual mesh filename=./meshes/MECANUM_WHEEL_M.dae
Joints:
- joint torso_0: origin xyz=0.0 0.0 0.2805 rpy=0.0 0.0 0.0 -> xyz=0.0 0.0 0.2965 rpy=0.0 0.0 0.0
- joint wheel_fl: axis 0 -1 0 -> 0 1 0; limit velocity=15.707963268 -> (none); origin xyz=0.228 0.265 0.1 rpy=0.0 0.0 0.0 -> xyz=0.243 0.245 0.076 rpy=0.0 0.0 0.0
- joint wheel_fr: axis 0 -1 0 -> 0 1 0; limit velocity=15.707963268 -> (none); origin xyz=0.228 -0.265 0.1 rpy=0.0 0.0 0.0 -> xyz=0.243 -0.245 0.076 rpy=0.0 0.0 0.0
- joint wheel_rl: axis 0 -1 0 -> 0 1 0; limit velocity=15.707963268 -> (none); origin xyz=0.228 0.265 0.1 rpy=0.0 0.0 0.0 -> xyz=-0.247 0.245 0.076 rpy=0.0 0.0 0.0
- joint wheel_rr: axis 0 -1 0 -> 0 1 0; limit velocity=15.707963268 -> (none); origin xyz=0.228 -0.265 0.1 rpy=0.0 0.0 0.0 -> xyz=-0.247 -0.245 0.076 rpy=0.0 0.0 0.0

Commit message: mecanum base 3D model modify and fix rby1_m urdf

File: models/rby1m/urdf/model.urdf (robot description, URDF)
Before this commit: robot RBY1_M, 36 links, 35 joints
Links:
- link wheel_fl_link: geometry visual mesh filename=./meshes/MECANUM_WHEEL_M.dae
- link wheel_rl_link: geometry visual mesh filename=./meshes/MECANUM_WHEEL.dae
