Commit message: feat: add nullspace joint target option for cartesian impedance control

File: models/rby1m/urdf/model_v1.3.urdf (robot description, URDF)
Before this commit: robot RBY1_M_v1.3, 34 links, 33 joints
Joints:
- joint END_left: origin xyz=0.0 0.0 -0.125 rpy=3.1415926535 0.0 0.0 -> xyz=0.0 0.0 -0.125 rpy=0 0.0 0.0
- joint END_right: origin xyz=0.0 0.0 -0.125 rpy=3.1415926535 0.0 0.0 -> xyz=0.0 0.0 -0.125 rpy=0 0.0 0.0
- joint gripper_finger_l1: origin xyz=0.0 0.0 0.0 rpy=3.1415926535 0.0 1.5707963268 -> xyz=0.0 0.0 0.0 rpy=0 0.0 1.5707963268
- joint gripper_finger_l2: origin xyz=0.0 0.0 0.0 rpy=3.1415926535 0.0 -1.5707963268 -> xyz=0.0 0.0 0.0 rpy=0 0.0 -1.5707963268
- joint gripper_finger_r1: origin xyz=0.0 0.0 0.0 rpy=3.1415926535 0.0 1.5707963268 -> xyz=0.0 0.0 0.0 rpy=0 0.0 1.5707963268
- joint gripper_finger_r2: origin xyz=0.0 0.0 0.0 rpy=3.1415926535 0.0 -1.5707963268 -> xyz=0.0 0.0 0.0 rpy=0 0.0 -1.5707963268
