Commit message: chore(model): add m v1.2

File: models/rby1m/urdf/model_v1.2.urdf (robot description, URDF)
Before this commit: robot RBY1_M_v1.3, 34 links, 33 joints
Links:
- link ee_left: mass 0.47470074 -> 0.46704998; geometry visual mesh filename=./meshes/EE_BODY.dae
- link ee_right: mass 0.47470074 -> 0.46704998; geometry visual mesh filename=./meshes/EE_BODY.dae
- link link_left_arm_4: mass 1.49373286 -> 0.42508710; geometry collision capsule colaffinity=1022 length=0.095000 radius=0.035; visual mesh filename=./meshes/LINK_18.dae
- link link_left_arm_5: mass 0.87163780 -> 1.60424243; geometry collision capsule colaffinity=1023 length=0.2213 radius=0.075; visual mesh filename=./meshes/LINK_19_v1.1.dae
- link link_left_arm_6: mass 0.74448182 -> 0.42751673; geometry visual mesh filename=./meshes/LINK_20_v1.1.dae
- link link_right_arm_4: mass 1.49373286 -> 0.42508710; geometry collision capsule colaffinity=30 coltype=256 length=0.095 radius=0.035; visual mesh filename=./meshes/LINK_11.dae
- link link_right_arm_5: mass 0.87163780 -> 1.60506693; geometry collision capsule colaffinity=31 coltype=512 length=0.2213 radius=0.075; visual mesh filename=./meshes/LINK_12_v1.1.dae
- link link_right_arm_6: mass 0.74448182 -> 0.42751673; geometry visual mesh filename=./meshes/LINK_13_v1.1.dae
Joints:
- removed joint END_left
- removed joint END_right
- added joint tool_left: type fixed, parent link_left_arm_6, child ee_left, origin xyz=0.0 0.0 -0.1261 rpy=0.0 0.0 0, axis 0 0 1
- added joint tool_right: type fixed, parent link_right_arm_6, child ee_right, origin xyz=0.0 0.0 -0.1261 rpy=0.0 0.0 0.0, axis 0 0 1
- joint gripper_finger_l1: axis 1 0 0 -> -1 0 0; limit lower=0.0 upper=0.05 effort=1000 velocity=0.05 -> lower=-0.05 upper=0 effort=1000 velocity=0.05; origin xyz=0.0 0.0 0.0 rpy=0 0.0 1.5707963268 -> xyz=0.003 0.0 -0.075 rpy=0.0 0.0 0.0
- joint gripper_finger_l2: axis -1 0 0 -> 1 0 0; limit lower=-0.05 upper=0.0 effort=1000 velocity=0.05 -> lower=0 upper=0.05 effort=1000 velocity=0.05; origin xyz=0.0 0.0 0.0 rpy=0 0.0 -1.5707963268 -> xyz=-0.003 0.0 -0.075 rpy=0.0 0.0 3.1415926535
- joint gripper_finger_r1: axis 1 0 0 -> -1 0 0; limit lower=0.0 upper=0.05 effort=1000 velocity=0.05 -> lower=-0.05 upper=0 effort=1000 velocity=0.05; origin xyz=0.0 0.0 0.0 rpy=0 0.0 1.5707963268 -> xyz=0.003 0.0 -0.075 rpy=0.0 0.0 0.0
- joint gripper_finger_r2: axis -1 0 0 -> 1 0 0; limit lower=-0.05 upper=0.0 effort=1000 velocity=0.05 -> lower=0 upper=0.05 effort=1000 velocity=0.05; origin xyz=0.0 0.0 0.0 rpy=0 0.0 -1.5707963268 -> xyz=-0.003 0.0 -0.075 rpy=0.0 0.0 3.1415926535
- joint left_arm_4: origin xyz=-0.031 0.0 -0.3095 rpy=0.0 0.0 0.0 -> xyz=-0.031 0.0 -0.256 rpy=0.0 0.0 0.0
- joint left_arm_5: limit lower=-0.8726646260 upper=0.8726646260 effort=10.0 velocity=6.283185308 -> lower=-1.570796327 upper=1.919862177 effort=10.0 velocity=6.283185308
- joint left_arm_6: axis 1 0 0 -> 0 0 1; limit lower=-1.5707963268 upper=1.5707963268 effort=8.0 velocity=2.094395102 -> lower=-2.705260340 upper=2.705260340 effort=8.0 velocity=2.094395102
- joint right_arm_4: origin xyz=-0.031 0.0 -0.3095 rpy=0.0 0.0 0.0 -> xyz=-0.031 0.0 -0.256 rpy=0.0 0.0 0.0
- joint right_arm_5: limit lower=-0.8726646260 upper=0.8726646260 effort=10.0 velocity=6.283185308 -> lower=-1.570796327 upper=1.919862177 effort=10.0 velocity=6.283185308
- joint right_arm_6: axis 1 0 0 -> 0 0 1; limit lower=-1.5707963268 upper=1.5707963268 effort=8.0 velocity=2.094395102 -> lower=-2.705260340 upper=2.705260340 effort=8.0 velocity=2.094395102
