Commit message: feat: add a v1.2 model

File: models/rby1a/urdf/model_v1.2.urdf (robot description, URDF)
Before this commit: robot RBY1_A_v1.2, 32 links, 31 joints
Links:
- link link_head_0: mass 0.07582110 -> 0.65731648; geometry visual mesh filename=./meshes/NECK_0.dae
- link link_head_1: mass 0.07450580 -> 0.70476502; geometry visual mesh filename=./meshes/NECK_1.dae
- link link_head_2: mass 0.03585374 -> 0.95262738; geometry visual mesh filename=./meshes/NECK_2.dae
- link link_torso_5: mass 12.59012341 -> 14.73283950
Joints:
- joint head_0: limit lower=-0.523 upper=0.523 effort=1000 velocity=3.14 -> lower=-1.57 upper=1.57 effort=1000 velocity=3.14; origin xyz=0.0 0.0 0.02 rpy=0.0 0.0 0.0 -> xyz=0.0 0.0 0.080 rpy=0.0 0.0 0.0
- joint head_1: limit lower=-0.35 upper=1.57 effort=1000 velocity=3.14 -> lower=-1.57 upper=1.57 effort=1000 velocity=3.14

Commit message: fix: model a v1.2 collisions for last links / model m mobile base kinematics param

File: models/rby1a/urdf/model_v1.2.urdf (robot description, URDF)
Before this commit: robot RBY1_A_v1.2, 32 links, 31 joints
Links:
- link link_left_arm_5: geometry collision capsule colaffinity=1023 length=0.2213 radius=0.075; visual mesh filename=./meshes/LINK_19_v1.1.dae
- link link_right_arm_5: geometry collision capsule colaffinity=31 coltype=512 length=0.2213 radius=0.075; visual mesh filename=./meshes/LINK_12_v1.1.dae
