Commit message: fix(models): update v1.2 link masses to measured values
Set the mass of the torso, both arms, grippers and head links in the
Model A and Model M v1.2 URDFs to the values weighed on the real robot.
Left and right arms use the same values. Inertia tensors and COM
origins are unchanged.

  link_torso_0..5     2.19 9.954 10.077 4.592 5.48 14.97
  link_*_arm_0..6     1.31 2.5 2.726 2.444 0.35 1.76 0.45
  ee_right/left       0.6
  ee_finger_*         0.04
  link_head_0..2      0.64 0.68 0.14

Co-Authored-By: Claude Opus 5.5 <noreply@anthropic.com>

File: models/rby1a/urdf/model_v1.2.urdf (robot description, URDF)
Before this commit: robot RBY1_A_v1.2, 32 links, 31 joints
Links:
- link ee_finger_l1: mass 0.03326999 -> 0.04
- link ee_finger_l2: mass 0.03326999 -> 0.04
- link ee_finger_r1: mass 0.03326999 -> 0.04
- link ee_finger_r2: mass 0.03326999 -> 0.04
- link ee_left: mass 0.46704998 -> 0.6
- link ee_right: mass 0.46704998 -> 0.6
- link link_head_0: mass 0.65731648 -> 0.64
- link link_head_1: mass 0.70476502 -> 0.68
- link link_head_2: mass 0.95262738 -> 0.14
- link link_left_arm_0: mass 1.26164242 -> 1.31
- link link_left_arm_1: mass 2.27287031 -> 2.5
- link link_left_arm_2: mass 2.46909439 -> 2.726
- link link_left_arm_3: mass 2.26099493 -> 2.444
- link link_left_arm_4: mass 0.42508710 -> 0.35
- link link_left_arm_5: mass 1.60506693 -> 1.76
- link link_left_arm_6: mass 0.42751673 -> 0.45
- link link_right_arm_0: mass 1.26164242 -> 1.31
- link link_right_arm_1: mass 2.27287031 -> 2.5
- link link_right_arm_2: mass 2.46909439 -> 2.726
- link link_right_arm_3: mass 2.26099493 -> 2.444
- link link_right_arm_4: mass 0.42508710 -> 0.35
- link link_right_arm_5: mass 1.60506693 -> 1.76
- link link_right_arm_6: mass 0.42751673 -> 0.45
- link link_torso_0: mass 2.24282123 -> 2.19
- link link_torso_1: mass 9.72162676 -> 9.954
- link link_torso_2: mass 9.21691850 -> 10.077
- link link_torso_3: mass 4.18679196 -> 4.592
- link link_torso_4: mass 4.45566276 -> 5.48
- link link_torso_5: mass 14.73283950 -> 14.97

File: models/rby1m/urdf/model_v1.2.urdf (robot description, URDF)
Before this commit: robot RBY1_M_v1.2, 34 links, 33 joints
Links:
- link ee_finger_l1: mass 0.03326999 -> 0.04
- link ee_finger_l2: mass 0.03326999 -> 0.04
- link ee_finger_r1: mass 0.03326999 -> 0.04
- link ee_finger_r2: mass 0.03326999 -> 0.04
- link ee_left: mass 0.46704998 -> 0.6
- link ee_right: mass 0.46704998 -> 0.6
- link link_head_0: mass 0.65731648 -> 0.64
- link link_head_1: mass 0.70476502 -> 0.68
- link link_head_2: mass 0.95262738 -> 0.14
- link link_left_arm_0: mass 1.26164242 -> 1.31
- link link_left_arm_1: mass 2.27287031 -> 2.5
- link link_left_arm_2: mass 2.46909439 -> 2.726
- link link_left_arm_3: mass 2.26099493 -> 2.444
- link link_left_arm_4: mass 0.42508710 -> 0.35
- link link_left_arm_5: mass 1.60506693 -> 1.76
- link link_left_arm_6: mass 0.42751673 -> 0.45
- link link_right_arm_0: mass 1.26164242 -> 1.31
- link link_right_arm_1: mass 2.27287031 -> 2.5
- link link_right_arm_2: mass 2.46909439 -> 2.726
- link link_right_arm_3: mass 2.26099493 -> 2.444
- link link_right_arm_4: mass 0.42508710 -> 0.35
- link link_right_arm_5: mass 1.60506693 -> 1.76
- link link_right_arm_6: mass 0.42751673 -> 0.45
- link link_torso_0: mass 2.24282123 -> 2.19
- link link_torso_1: mass 9.72162676 -> 9.954
- link link_torso_2: mass 9.21691850 -> 10.077
- link link_torso_3: mass 4.18679196 -> 4.592
- link link_torso_4: mass 4.45566276 -> 5.48
- link link_torso_5: mass 14.73283950 -> 14.97
