Commit message: feat: add model A v1.1

File: models/rby1a/urdf/model_v1.0.urdf (robot description, URDF)
Before this commit: robot RBY1_A_v1.0, 34 links, 33 joints
Joints:
- joint left_arm_0: axis 0 1 0 -> 0.0 0.93969262 0.34202014; origin xyz=0.0 0.220 0.080073452  rpy=0.349065850  0.0 0.0 -> xyz=0.0 0.220 0.080073452  rpy=0.0 0.0 0.0
- joint left_arm_1: origin xyz=0.0 0.0 0.0 rpy=-0.349065850 0.0 0.0 -> xyz=0.0 0.0 0.0 rpy=0.0 0.0 0.0
- joint right_arm_0: axis 0 1 0 -> 0.0 0.93969262 -0.34202014; origin xyz=0.0 -0.220 0.080073451539  rpy=-0.349065850  0.0 0.0 -> xyz=0.0 -0.220 0.080073451539  rpy=0.0 0.0 0.0
- joint right_arm_1: origin xyz=0.0 0.0 0.0 rpy=0.349065850 0.0 0.0 -> xyz=0.0 0.0 0.0 rpy=0.0 0.0 0.0

File: models/rby1a/urdf/model_v1.1.urdf (robot description, URDF)
Before this commit: robot RBY1_A_v1.0, 34 links, 33 joints
Links:
- removed link FT_sensor_L
- removed link FT_sensor_R
- link link_left_arm_5: mass 1.44264795 -> 1.60424243; geometry collision capsule colaffinity=1023 length=0.25 radius=0.075; visual mesh filename=./meshes/LINK_19_v1.1.dae
- link link_left_arm_6: mass 0.21137279 -> 0.42751673; geometry visual mesh filename=./meshes/LINK_20_v1.1.dae
- link link_right_arm_5: mass 1.59194395 -> 1.60506693; geometry collision capsule colaffinity=31 coltype=512 length=0.25 radius=0.075; visual mesh filename=./meshes/LINK_12_v1.1.dae
- link link_right_arm_6: mass 0.21137279 -> 0.42751673; geometry visual mesh filename=./meshes/LINK_13_v1.1.dae
Joints:
- removed joint FT_Sensor_END_left
- removed joint FT_Sensor_END_right
- joint gripper_finger_l1: origin xyz=0.003 0.0 -0.073 rpy=0.0 0.0 0.0 -> xyz=0.003 0.0 -0.075 rpy=0.0 0.0 0.0
- joint gripper_finger_l2: origin xyz=-0.003 0.0 -0.073 rpy=0.0 0.0 3.1415926535 -> xyz=-0.003 0.0 -0.075 rpy=0.0 0.0 3.1415926535
- joint gripper_finger_r1: origin xyz=0.003 0.0 -0.073 rpy=0.0 0.0 0.0 -> xyz=0.003 0.0 -0.075 rpy=0.0 0.0 0.0
- joint gripper_finger_r2: origin xyz=-0.003 0.0 -0.073 rpy=0.0 0.0 3.1415926535 -> xyz=-0.003 0.0 -0.075 rpy=0.0 0.0 3.1415926535
- joint left_arm_0: axis 0 1 0 -> 0.0 0.93969262 0.34202014; origin xyz=0.0 0.220 0.080073452  rpy=0.349065850  0.0 0.0 -> xyz=0.0 0.220 0.080073452  rpy=0.0 0.0 0.0
- joint left_arm_1: origin xyz=0.0 0.0 0.0 rpy=-0.349065850 0.0 0.0 -> xyz=0.0 0.0 0.0 rpy=0.0 0.0 0.0
- joint right_arm_0: axis 0 1 0 -> 0.0 0.93969262 -0.34202014; origin xyz=0.0 -0.220 0.080073451539  rpy=-0.349065850  0.0 0.0 -> xyz=0.0 -0.220 0.080073451539  rpy=0.0 0.0 0.0
- joint right_arm_1: origin xyz=0.0 0.0 0.0 rpy=0.349065850 0.0 0.0 -> xyz=0.0 0.0 0.0 rpy=0.0 0.0 0.0
- joint tool_left: child FT_sensor_L -> ee_left; origin xyz=0.0 0.0 -0.1087 rpy=0.0 0.0 0 -> xyz=0.0 0.0 -0.1261 rpy=0.0 0.0 0
- joint tool_right: child FT_sensor_R -> ee_right; origin xyz=0.0 0.0 -0.1087 rpy=0.0 0.0 0.0 -> xyz=0.0 0.0 -0.1261 rpy=0.0 0.0 0.0

Commit message: fix(urdf): fix inertia values for left/right arm URDFs
Adjusted inertia matrix and origin xyz for both arms to correct mirroring issue.

File: models/rby1a/urdf/model_v1.0.urdf (robot description, URDF)
Before this commit: robot RBY1_A_v1.0, 34 links, 33 joints
Links:
- link link_left_arm_1: mass 1.88138658 -> 2.27287031
- link link_left_arm_2: mass 2.35634437 -> 2.46909439
- link link_left_arm_3: mass 2.00905891 -> 2.26099493
- link link_left_arm_5: mass 1.44264795 -> 1.59194395

File: models/rby1a/urdf/model_v1.1.urdf (robot description, URDF)
Before this commit: robot RBY1_A_v1.1, 32 links, 31 joints
Links:
- link link_left_arm_1: mass 1.88138658 -> 2.27287031
- link link_left_arm_2: mass 2.35634437 -> 2.46909439
- link link_left_arm_3: mass 2.00905891 -> 2.26099493
- link link_left_arm_5: mass 1.60424243 -> 1.60506693; geometry collision capsule colaffinity=1023 length=0.2213 radius=0.075; visual mesh filename=./meshes/LINK_19_v1.1.dae
- link link_right_arm_5: geometry collision capsule colaffinity=31 coltype=512 length=0.2213 radius=0.075; visual mesh filename=./meshes/LINK_12_v1.1.dae

File: models/rby1a/urdf/model_v1.2.urdf (robot description, URDF)
Before this commit: robot RBY1_A_v1.2, 32 links, 31 joints
Links:
- link link_left_arm_1: mass 1.88138658 -> 2.27287031
- link link_left_arm_2: mass 2.35634437 -> 2.46909439
- link link_left_arm_3: mass 2.00905891 -> 2.26099493
- link link_left_arm_5: mass 1.60424243 -> 1.60506693

File: models/rby1m/urdf/model.urdf (robot description, URDF)
Before this commit: robot RBY1_M, 36 links, 35 joints
Links:
- link link_left_arm_1: mass 1.88138658 -> 2.27287031
- link link_left_arm_2: mass 2.35634437 -> 2.46909439
- link link_left_arm_3: mass 2.00905891 -> 2.26099493
- link link_left_arm_5: mass 1.44264795 -> 1.59194395

File: models/rby1m/urdf/model_v1.1.urdf (robot description, URDF)
Before this commit: robot RBY1_M_v1.1, 34 links, 33 joints
Links:
- link link_left_arm_1: mass 1.88138658 -> 2.27287031
- link link_left_arm_2: mass 2.35634437 -> 2.46909439
- link link_left_arm_3: mass 2.00905891 -> 2.26099493
- link link_left_arm_5: mass 1.60424243 -> 1.60506693

File: models/rby1m/urdf/model_v1.2.urdf (robot description, URDF)
Before this commit: robot RBY1_M_v1.2, 34 links, 33 joints
Links:
- link link_left_arm_1: mass 1.88138658 -> 2.27287031
- link link_left_arm_2: mass 2.35634437 -> 2.46909439
- link link_left_arm_3: mass 2.00905891 -> 2.26099493
- link link_left_arm_5: mass 1.60424243 -> 1.60506693

File: models/rby1m/urdf/model_v1.3.urdf (robot description, URDF)
Before this commit: robot RBY1_M_v1.3, 34 links, 33 joints
Links:
- link link_left_arm_1: mass 1.88138658 -> 2.27287031
- link link_left_arm_2: mass 2.35634437 -> 2.46909439
- link link_left_arm_3: mass 2.00905891 -> 2.26099493
Joints:
- joint END_left: origin xyz=0.0 0.0 -0.125 rpy=0 0.0 0.0 -> xyz=0.0 0.0 -0.125 rpy=3.1415926535 0.0 0.0
- joint END_right: origin xyz=0.0 0.0 -0.125 rpy=0 0.0 0.0 -> xyz=0.0 0.0 -0.125 rpy=3.1415926535 0.0 0.0
- joint gripper_finger_l1: origin xyz=0.0 0.0 0.0 rpy=0 0.0 1.5707963268 -> xyz=0.0 0.0 0.0 rpy=3.1415926535 0.0 1.5707963268
- joint gripper_finger_l2: origin xyz=0.0 0.0 0.0 rpy=0 0.0 -1.5707963268 -> xyz=0.0 0.0 0.0 rpy=3.1415926535 0.0 -1.5707963268
- joint gripper_finger_r1: origin xyz=0.0 0.0 0.0 rpy=0 0.0 1.5707963268 -> xyz=0.0 0.0 0.0 rpy=3.1415926535 0.0 1.5707963268
- joint gripper_finger_r2: origin xyz=0.0 0.0 0.0 rpy=0 0.0 -1.5707963268 -> xyz=0.0 0.0 0.0 rpy=3.1415926535 0.0 -1.5707963268
