Commit message: fix(model.urdf): Change velocity limits for urdf torso_0, torso_1, and left_arm_5
Changed velocity limits for torso_0 and torso_1 from 3.14159265 rad/s to 2.09439510 rad/s (equivalent to 180deg/s to 120deg/s), and for left_arm_5 from 30.14159265 rad/s to 3.14159265 rad/s.

File: models/rby1a/urdf/model.urdf (robot description, URDF)
Before this commit: robot RB_Y1_V1.0.1, 34 links, 33 joints
Joints:
- joint left_arm_5: limit lower=-1.74532925 upper=2.00712864 effort=1000.0 velocity=30.14159265 -> lower=-1.74532925 upper=2.00712864 effort=1000.0 velocity=3.14159265
- joint torso_0: limit lower=-0.34906585 upper=0.34906585 effort=1000.0 velocity=3.14159265 -> lower=-0.34906585 upper=0.34906585 effort=1000.0 velocity=2.09439510
- joint torso_1: limit lower=-1.04719755 upper=1.52173048 effort=1000.0 velocity=3.14159265 -> lower=-1.04719755 upper=1.52173048 effort=1000.0 velocity=2.09439510

Commit message: fix: align mobility SE2 and joint velocity direction with RPC program for simulator consistency

File: models/rby1a/urdf/model.urdf (robot description, URDF)
Before this commit: robot RB_Y1_V1.0.1, 34 links, 33 joints
Joints:
- joint left_wheel: axis 0 1 0 -> 0 -1 0
- joint right_wheel: axis 0 1 0 -> 0 -1 0

Commit message: feat: expand gripper tip collision area

File: models/rby1a/urdf/model.urdf (robot description, URDF)
Before this commit: robot RB_Y1_V1.0.1, 34 links, 33 joints
Links:
- link link_left_arm_5: geometry collision capsule colaffinity=1023 length=0.25 radius=0.075; visual mesh filename=./meshes/LINK_19.dae
- link link_right_arm_5: geometry collision capsule colaffinity=31 coltype=512 length=0.25 radius=0.075; visual mesh filename=./meshes/LINK_12.dae

Commit message: fix: make joint values realistic (#33)

File: models/rby1a/urdf/model.urdf (robot description, URDF)
Before this commit: robot RB_Y1_V1.0.1, 34 links, 33 joints
Joints:
- joint left_arm_0: limit lower=-2.35619449 upper=2.35619449 effort=1000.0 velocity=3.14159265 -> lower=-3.141592654 upper=3.141592654 effort=70.0 velocity=3.141592654
- joint left_arm_1: limit lower=-0.05 upper=3.14159265 effort=1000.0 velocity=3.14159265 -> lower=-0.017453293 upper=3.141592654 effort=70.0 velocity=3.141592654
- joint left_arm_2: limit lower=-2.09439510 upper=2.09439510 effort=1000.0 velocity=3.14159265 -> lower=-3.141592654 upper=3.141592654 effort=70.0 velocity=3.141592654
- joint left_arm_3: limit lower=-2.61799388 upper=0.01 effort=1000.0 velocity=3.14159265 -> lower=-2.617993878 upper=0.017453293 effort=40.0 velocity=3.141592654
- joint left_arm_4: limit lower=-6.28318531 upper=6.28318531 effort=1000.0 velocity=3.14159265 -> lower=-3.141592654 upper=3.141592654 effort=10.0 velocity=6.283185308
- joint left_arm_5: limit lower=-1.74532925 upper=2.00712864 effort=1000.0 velocity=3.14159265 -> lower=-1.570796327 upper=1.919862177 effort=10.0 velocity=6.283185308
- joint left_arm_6: limit lower=-2.96705973 upper=2.96705973 effort=1000.0 velocity=3.14159265 -> lower=-2.792526803 upper=2.792526803 effort=8.0 velocity=2.094395102
- joint left_wheel: limit velocity=3.14159265 -> velocity=15.707963268
- joint right_arm_0: limit lower=-2.35619449 upper=2.35619449 effort=1000.0 velocity=3.14159265 -> lower=-3.141592654 upper=3.141592654 effort=70.0 velocity=3.141592654
- joint right_arm_1: limit lower=-3.14159265 upper=0.05 effort=1000.0 velocity=3.14159265 -> lower=-3.141592654 upper=0.017453293 effort=70.0 velocity=3.141592654
- joint right_arm_2: limit lower=-2.09439510 upper=2.09439510 effort=1000.0 velocity=3.14159265 -> lower=-3.141592654 upper=3.141592654 effort=70.0 velocity=3.141592654
- joint right_arm_3: limit lower=-2.61799388 upper=0.01 effort=1000.0 velocity=3.14159265 -> lower=-2.617993878 upper=0.017453293 effort=40.0 velocity=3.141592654
- joint right_arm_4: limit lower=-6.28318531 upper=6.28318531 effort=1000.0 velocity=3.14159265 -> lower=-3.141592654 upper=3.141592654 effort=10.0 velocity=6.283185308
- joint right_arm_5: limit lower=-1.74532925 upper=2.00712864 effort=1000.0 velocity=3.14159265 -> lower=-1.570796327 upper=1.919862177 effort=10.0 velocity=6.283185308
- joint right_arm_6: limit lower=-2.96705973 upper=2.96705973 effort=1000.0 velocity=3.14159265 -> lower=-2.792526803 upper=2.792526803 effort=8.0 velocity=2.094395102
- joint right_wheel: limit velocity=3.14159265 -> velocity=15.707963268
- joint torso_0: limit lower=-0.34906585 upper=0.34906585 effort=1000.0 velocity=2.09439510 -> lower=-0.261799388 upper=0.261799388 effort=270.0 velocity=2.09439510
- joint torso_1: limit lower=-1.04719755 upper=1.52173048 effort=1000.0 velocity=2.09439510 -> lower=-0.523598776 upper=1.570796327 effort=270.0 velocity=2.09439510
- joint torso_2: limit lower=-2.478367 upper=1.570796 effort=1000.0 velocity=3.14159265 -> lower=-2.617993878 upper=1.570796327 effort=270.0 velocity=2.09439510
- joint torso_3: limit lower=-0.78539816 upper=1.57079633 effort=1000.0 velocity=3.14159265 -> lower=-0.785398163 upper=0.785398163 effort=120.0 velocity=3.141592654
- joint torso_4: limit lower=-0.52359878 upper=0.52359878 effort=1000.0 velocity=3.14159265 -> lower=-0.523598776 upper=0.523598776 effort=120.0 velocity=3.141592654
- joint torso_5: limit lower=-1.57079633 upper=1.57079633 effort=1000.0 velocity=3.14159265 -> lower=-2.35619449 upper=2.35619449 effort=120.0 velocity=3.141592654

Commit message: feat: update joint limit

File: models/rby1a/urdf/model.urdf (robot description, URDF)
Before this commit: robot RB_Y1_V1.0.1, 34 links, 33 joints
Joints:
- joint torso_3: limit lower=-0.785398163 upper=0.785398163 effort=120.0 velocity=3.141592654 -> lower=-0.785398163 upper=1.04719755 effort=120.0 velocity=3.141592654

Commit message: feat(model.urdf): update joint limit(torso_3)

File: models/rby1a/urdf/model.urdf (robot description, URDF)
Before this commit: robot RB_Y1_V1.0.1, 34 links, 33 joints
Joints:
- joint torso_3: limit lower=-0.785398163 upper=1.04719755 effort=120.0 velocity=3.141592654 -> lower=-0.785398163 upper=1.570796327 effort=120.0 velocity=3.141592654

Commit message: fix: adjust wrist yaw2 range of motion in model.urdf for A, T5, and M models (#85)

File: models/rby1a/urdf/model.urdf (robot description, URDF)
Before this commit: robot RB_Y1_V1.0.1, 34 links, 33 joints
Joints:
- joint left_arm_6: limit lower=-2.792526803 upper=2.792526803 effort=8.0 velocity=2.094395102 -> lower=-2.705260340 upper=2.705260340 effort=8.0 velocity=2.094395102
- joint right_arm_6: limit lower=-2.792526803 upper=2.792526803 effort=8.0 velocity=2.094395102 -> lower=-2.705260340 upper=2.705260340 effort=8.0 velocity=2.094395102

File: models/rby1m/urdf/model.urdf (robot description, URDF)
Before this commit: robot RB_Y1M, 36 links, 35 joints
Joints:
- joint left_arm_6: limit lower=-2.792526803 upper=2.792526803 effort=8.0 velocity=2.094395102 -> lower=-2.705260340 upper=2.705260340 effort=8.0 velocity=2.094395102
- joint right_arm_6: limit lower=-2.792526803 upper=2.792526803 effort=8.0 velocity=2.094395102 -> lower=-2.705260340 upper=2.705260340 effort=8.0 velocity=2.094395102

File: models/rby1t5/urdf/model.urdf (robot description, URDF)
Before this commit: robot RB_Y1_V1.0.1, 34 links, 33 joints
Joints:
- joint left_arm_6: limit lower=-2.792526803 upper=2.792526803 effort=8.0 velocity=2.094395102 -> lower=-2.705260340 upper=2.705260340 effort=8.0 velocity=2.094395102
- joint right_arm_6: limit lower=-2.792526803 upper=2.792526803 effort=8.0 velocity=2.094395102 -> lower=-2.705260340 upper=2.705260340 effort=8.0 velocity=2.094395102

Commit message: fix: correct shoulder 0 link frame orientation in rby1a urdf model

File: models/rby1a/urdf/model.urdf (robot description, URDF)
Before this commit: robot RBY1_A_v1.0, 34 links, 33 joints
Joints:
- joint left_arm_0: axis 0 1 0 -> 0.0 0.93969262 0.34202014; origin xyz=0.0 0.220 0.080073452  rpy=0.349065850  0.0 0.0 -> xyz=0.0 0.220 0.080073452  rpy=0.0 0.0 0.0
- joint left_arm_1: origin xyz=0.0 0.0 0.0 rpy=-0.349065850 0.0 0.0 -> xyz=0.0 0.0 0.0 rpy=0.0 0.0 0.0
- joint right_arm_0: axis 0 1 0 -> 0.0 0.93969262 -0.34202014; origin xyz=0.0 -0.220 0.080073451539  rpy=-0.349065850  0.0 0.0 -> xyz=0.0 -0.220 0.080073451539  rpy=0.0 0.0 0.0
- joint right_arm_1: origin xyz=0.0 0.0 0.0 rpy=0.349065850 0.0 0.0 -> xyz=0.0 0.0 0.0 rpy=0.0 0.0 0.0

Commit message: fix(urdf): fix inertia values for left/right arm URDFs
Adjusted inertia matrix and origin xyz for both arms to correct mirroring issue.

File: models/rby1a/urdf/model.urdf (robot description, URDF)
Before this commit: robot RBY1_A_v1.0, 34 links, 33 joints
Links:
- link link_left_arm_1: mass 1.88138658 -> 2.27287031
- link link_left_arm_2: mass 2.35634437 -> 2.46909439
- link link_left_arm_3: mass 2.00905891 -> 2.26099493
- link link_left_arm_5: mass 1.44264795 -> 1.59194395
